Commit message: Removed underscore after prefix.

File: ridgeback_description/urdf/accessories/sick_lms1xx_mount.urdf.xacro (robot description, xacro)
@@ -32,5 +32,5 @@
       <origin xyz="${location * 0.3999} 0 0.2337" rpy="0 0 ${PI/2 - (location * PI/2)}" />
       <parent link="chassis_link" />
-      <child link="${prefix}_laser" />
+      <child link="${prefix}laser" />
     </joint>
   </xacro:macro>
