Commit message: Update description with some rough measurements.

File: ridgeback_description/urdf/ridgeback.urdf.xacro (robot description, xacro)
@@ -2,13 +2,12 @@
 <robot name="ridgeback" xmlns:xacro="http://www.ros.org/wiki/xacro">
   <xacro:property name="PI" value="3.1415926535897931" />
-  <xacro:property name="wheelbase" value="0.262" />
-  <xacro:property name="track" value="0.37559" />
-  <xacro:property name="wheel_vertical_offset" value="0.0345" />
-  <xacro:property name="footprint_vertical_offset" value="-0.0655" />
-  <xacro:property name="wheel_radius" value="0.098" />
-  <xacro:property name="wheel_width" value="0.040" />
-  <xacro:property name="chassis_length" value="0.420" />
-  <xacro:property name="chassis_width" value="0.310" />
-  <xacro:property name="chassis_height" value="0.184" />
+  <xacro:property name="wheelbase" value="0.610" />
+  <xacro:property name="track" value="0.622" />
+  <xacro:property name="wheel_vertical_offset" value="0.05" />
+  <xacro:property name="wheel_radius" value="0.1518" />
+  <xacro:property name="wheel_width" value="0.0471" />
+  <xacro:property name="chassis_length" value="0.927" />
+  <xacro:property name="chassis_width" value="0.787" />
+  <xacro:property name="chassis_height" value="0.216" />
   <xacro:property name="dummy_inertia" value="1e-09"/>
   <xacro:property name="mount_spacing" value="0.120" />
@@ -22,5 +21,6 @@
         <origin xyz="0 0 0" rpy="${PI/2} 0 0"/>
         <geometry>
-          <mesh filename="package://ridgeback_description/meshes/ridgeback-wheel.stl"/>
+          <!--<mesh filename="package://ridgeback_description/meshes/ridgeback-wheel.stl"/> -->
+          <cylinder radius="${wheel_radius}" length="${wheel_width}"/>
         </geometry>
         <material name="black" />
@@ -89,7 +89,7 @@
   <link name="chassis_link">
     <visual>
-      <origin xyz="0 0 ${footprint_vertical_offset}" rpy="${PI/2} 0 ${PI/2}"/>
+      <origin xyz="0 0 ${chassis_height/2}"/>
       <geometry>
-        <mesh filename="package://ridgeback_description/meshes/ridgeback-base.stl"/>
+        <box size="${chassis_length} ${chassis_width} ${chassis_height}"/>
       </geometry>
       <material name="dark_grey" />
@@ -101,16 +101,14 @@
       </geometry>
     </collision>
-    <inertial>
-      <!-- Center of mass -->
+    <!--<inertial>
       <origin xyz="0.012  0.002 0.067" rpy="0 0 0"/>
       <mass value="16.523"/>
-      <!-- Moments of inertia: ( chassis without wheels ) -->
       <inertia
         ixx="0.3136" ixy="-0.0008" ixz="0.0164"
         iyy="0.3922" iyz="-0.0009"
         izz="0.4485"/>
-      </inertial>
+      </inertial>-->
   </link>
-  <link name="fenders_link">
+  <!--<link name="fenders_link">
     <visual>
       <origin xyz="0 0 ${footprint_vertical_offset}" rpy="${PI/2} 0 ${PI/2}"/>
@@ -124,5 +122,5 @@
     <parent link="chassis_link" />
     <child link="fenders_link" />
-  </joint>
+  </joint>-->
   <!-- TODO: Make this internal_imu_link or something, and use a mixed-in xacro
        to supply the joint between it and imu_link. This is important so that imu_link
@@ -140,44 +138,11 @@
     <child link="imu_link" />
   </joint>
-  <!-- TODO: Same note as applies to imu_link -->
-  <link name="navsat_link">
-    <visual>
-      <geometry>
-        <cylinder radius="0.026" length="0.016" />
-      </geometry>
-      <origin xyz="0 0 0.008" />
-      <material name="black" />
-    </visual>
-  </link>
-  <joint name="navsat_joint" type="fixed">
-    <parent link="chassis_link" />
-    <child link="navsat_link" />
-    <origin xyz="-0.180 0.126 0.1815" />
-  </joint>
-  <link name="mid_mount"></link>
-  <joint name="mid_mount_joint" type="fixed">
-    <parent link="chassis_link" />
-    <child link="mid_mount" />
-    <origin xyz="0 0 ${chassis_height}" />
-  </joint>
-  <link name="rear_mount"></link>
-  <joint name="rear_mount_joint" type="fixed">
-    <parent link="mid_mount" />
-    <child link="rear_mount" />
-    <origin xyz="${-mount_spacing} 0 0" />
-  </joint>
-  <link name="front_mount"></link>
-  <joint name="front_mount_joint" type="fixed">
-    <parent link="mid_mount" />
-    <child link="front_mount" />
-    <origin xyz="${mount_spacing} 0 0" />
-  </joint>
   <!-- Bring in simulation data for Gazebo. -->
-  <xacro:include filename="ridgeback.gazebo" />
+  <!--<xacro:include filename="ridgeback.gazebo" />-->
   <!-- Optional standard accessories, including their simulation data. The rendering
        of these into the final description is controlled by optenv variables, which
        default each one to off.-->
-  <xacro:include filename="accessories.urdf.xacro" />
+  <!--<xacro:include filename="accessories.urdf.xacro" />-->
   <!-- Optional custom includes. -->
-  <xacro:include filename="$(optenv RIDGEBACK_URDF_EXTRAS empty.urdf)" />
+  <!--<xacro:include filename="$(optenv RIDGEBACK_URDF_EXTRAS empty.urdf)" />-->
 </robot>

Commit message: In-progress.

File: ridgeback_description/urdf/ridgeback.urdf.xacro (robot description, xacro)
@@ -31,13 +31,4 @@
           <cylinder radius="${wheel_radius}" length="${wheel_width}"/>
         </geometry>
-        <friction>
-          <ode>
-            <fdir1>0.707107 ${y_friction} 0.000000</fdir1>
-            <mu1>0.0001</mu1>
-            <mu2>1000</mu2>
-            <slip1>1000</slip1>
-            <slip2>0.0001</slip2>
-          </ode>
-        </friction>
       </collision>
       <inertial>
@@ -52,4 +43,13 @@
     <gazebo reference="${prefix}_wheel_link">
       <material>Gazebo/DarkGrey</material>
+      <friction>
+        <ode>
+          <fdir1>0.707107 ${y_friction} 0.000000</fdir1>
+          <mu1>0.0001</mu1>
+          <mu2>1000</mu2>
+          <slip1>1000</slip1>
+          <slip2>0.0001</slip2>
+        </ode>
+      </friction>
     </gazebo>
     <joint name="${prefix}_wheel" type="continuous">
@@ -101,5 +101,5 @@
       </geometry>
     </collision>
-    <!--<inertial>
+    <inertial>
       <origin xyz="0.012  0.002 0.067" rpy="0 0 0"/>
       <mass value="16.523"/>
@@ -108,5 +108,5 @@
         iyy="0.3922" iyz="-0.0009"
         izz="0.4485"/>
-      </inertial>-->
+    </inertial>
   </link>
   <!--<link name="fenders_link">

Commit message: Remove fenders.

File: ridgeback_description/urdf/ridgeback.urdf.xacro (robot description, xacro)
@@ -110,17 +110,4 @@
     </inertial>
   </link>
-  <!--<link name="fenders_link">
-    <visual>
-      <origin xyz="0 0 ${footprint_vertical_offset}" rpy="${PI/2} 0 ${PI/2}"/>
-      <geometry>
-        <mesh filename="package://ridgeback_description/meshes/ridgeback-fenders.stl"/>
-      </geometry>
-      <material name="yellow" />
-    </visual>
-  </link>
-  <joint name="fenders_joint" type="fixed">
-    <parent link="chassis_link" />
-    <child link="fenders_link" />
-  </joint>-->
   <!-- TODO: Make this internal_imu_link or something, and use a mixed-in xacro
        to supply the joint between it and imu_link. This is important so that imu_link

Commit message: WIP URDF, waiting on meshes with origin in geometric centre.

File: ridgeback_description/urdf/ridgeback.urdf.xacro (robot description, xacro)
@@ -5,9 +5,12 @@
   <xacro:property name="track" value="0.622" />
   <xacro:property name="wheel_vertical_offset" value="0.05" />
-  <xacro:property name="wheel_radius" value="0.1518" />
+  <xacro:property name="wheel_radius" value="0.0759" />
   <xacro:property name="wheel_width" value="0.0471" />
   <xacro:property name="chassis_length" value="0.927" />
   <xacro:property name="chassis_width" value="0.787" />
   <xacro:property name="chassis_height" value="0.216" />
+  <xacro:property name="cover_offset" value="0.240" />
+  <xacro:property name="top_offset" value="0.05" />
+  <!-- Need to verify values above -->
   <xacro:property name="dummy_inertia" value="1e-09"/>
   <xacro:property name="mount_spacing" value="0.120" />
@@ -16,11 +19,10 @@
   <material name="yellow"><color rgba="0.8 0.8 0.0 1.0" /></material>
   <material name="black"><color rgba="0.15 0.15 0.15 1.0" /></material>
-  <xacro:macro name="wheel" params="prefix y_friction *joint_pose">
-    <link name="${prefix}_wheel_link">
+  <xacro:macro name="wheel" params="prefix side y_friction *joint_pose">
+    <link name="${prefix}_${side}_wheel_link">
       <visual>
         <origin xyz="0 0 0" rpy="${PI/2} 0 0"/>
         <geometry>
-          <!--<mesh filename="package://ridgeback_description/meshes/ridgeback-wheel.stl"/> -->
-          <cylinder radius="${wheel_radius}" length="${wheel_width}"/>
+          <mesh filename="package://ridgeback_description/meshes/wheel.stl"/>
         </geometry>
         <material name="black" />
@@ -41,5 +43,5 @@
       </inertial>
     </link>
-    <gazebo reference="${prefix}_wheel_link">
+    <gazebo reference="${prefix}_${side}_wheel_link">
       <material>Gazebo/DarkGrey</material>
       <friction>
@@ -53,7 +55,7 @@
       </friction>
     </gazebo>
-    <joint name="${prefix}_wheel" type="continuous">
-      <parent link="chassis_link"/>
-      <child link="${prefix}_wheel_link" />
+    <joint name="${prefix}_${side}_wheel" type="continuous">
+      <parent link="${prefix}_rocker_link"/>
+      <child link="${prefix}_${side}_wheel_link" />
       <xacro:insert_block name="joint_pose" />
       <axis xyz="0 1 0" />
@@ -64,21 +66,54 @@
         <hardwareInterface>VelocityJointInterface</hardwareInterface>
       </joint>
-      <actuator name="${prefix}_actuator">
+      <actuator name="${prefix}_${side}_actuator">
         <mechanicalReduction>1</mechanicalReduction>
       </actuator>
     </transmission>
   </xacro:macro>
-  <xacro:wheel prefix="front_left" y_friction="-0.707107">
-    <origin xyz="${wheelbase/2} ${track/2} ${wheel_vertical_offset}" rpy="0 0 0" />
+<xacro:macro name="rocker" params="prefix joint_type wheel_location *joint_limits">
+  <link name="${prefix}_rocker_link">
+    <visual>
+      <origin xyz="0 0 0" rpy="0 0 0"/>
+      <geometry>
+        <mesh filename="package://ridgeback_description/meshes/rocker.stl"/>
+      </geometry>
+      <material name="black" />
+    </visual>
+    <collision>
+      <origin xyz="0 0 0" rpy="0 0 0"/>
+      <geometry>
+        <box size="${wheelbase} ${track} 0"/>
+      </geometry>
+    </collision>
+  </link>
+  <joint name="${prefix}_rocker" type="${joint_type}">
+    <parent link="axle_link"/>
+    <child link="${prefix}_rocker_link" />
+    <origin xyz="0 0 0" rpy="0 0 0" />
+    <axis xyz="1 0 0" />
+    <xacro:insert_block name="joint_limits" />
+  </joint>
+  <transmission name="${prefix}_rocker_trans">
+    <type>transmission_interface/SimpleTransmission</type>
+    <joint name="${prefix}_rocker">
+      <hardwareInterface>VelocityJointInterface</hardwareInterface>
+    </joint>
+    <actuator name="${prefix}_actuator">
+      <mechanicalReduction>1</mechanicalReduction>
+    </actuator>
+  </transmission>
+  <xacro:wheel prefix="${prefix}" side="left" y_friction="-0.707107">
+    <origin xyz="${wheel_location*wheelbase/2} ${track/2} ${wheel_vertical_offset}" rpy="0 0 0" />
   </xacro:wheel>
-  <xacro:wheel prefix="front_right" y_friction="0.707107">
-    <origin xyz="${wheelbase/2} ${-track/2} ${wheel_vertical_offset}" rpy="0 0 0" />
+  <xacro:wheel prefix="${prefix}" side="right" y_friction="0.707107">
+    <origin xyz="${wheel_location*wheelbase/2} ${-track/2} ${wheel_vertical_offset}" rpy="0 0 0" />
   </xacro:wheel>
-  <xacro:wheel prefix="rear_left" y_friction="0.707107">
-    <origin xyz="${-wheelbase/2} ${track/2} ${wheel_vertical_offset}" rpy="0 0 0" />
-  </xacro:wheel>
-  <xacro:wheel prefix="rear_right" y_friction="-0.707107">
-    <origin xyz="${-wheelbase/2} ${-track/2} ${wheel_vertical_offset}" rpy="0 0 0" />
-  </xacro:wheel>
+</xacro:macro>
+<xacro:rocker prefix="front" joint_type="revolute" wheel_location="1" >
+  <limit lower="-0.2" upper="0.2" effort="0" velocity="0" />
+</xacro:rocker>
+<xacro:rocker prefix="rear" joint_type="fixed" wheel_location="-1" >
+  <limit effort="0" velocity="0" />
+</xacro:rocker>
   <link name="base_link"></link>
   <joint name="base_link_joint" type="fixed">
@@ -89,12 +124,12 @@
   <link name="chassis_link">
     <visual>
-      <origin xyz="0 0 ${chassis_height/2}"/>
-      <geometry>
-        <box size="${chassis_length} ${chassis_width} ${chassis_height}"/>
-      </geometry>
-      <material name="dark_grey" />
+      <origin xyz="0 0 0" rpy=" 0 0 0" />
+      <geometry>
+        <mesh filename="package://ridgeback_description/meshes/body.stl"/>
+      </geometry>
+      <material name="black" />
     </visual>
     <collision>
-      <origin xyz="0 0 ${chassis_height/2}"/>
+      <origin xyz="0 0 0"/>
       <geometry>
         <box size="${chassis_length} ${chassis_width} ${chassis_height}"/>
@@ -109,4 +144,60 @@
         izz="0.4485"/>
     </inertial>
+  </link>
+<joint name="front_cover_link_joint" type="fixed">
+  <origin xyz="0 0 0" rpy="0 0 0" />
+  <parent link="chassis_link"/>
+  <child link="front_cover_link" />
+</joint>
+  <link name="front_cover_link">
+    <visual>
+      <origin xyz="${cover_offset} ${-chassis_width/2} 0" rpy=" 0 0 0" />
+      <geometry>
+        <mesh filename="package://ridgeback_description/meshes/end-cover.stl"  scale="0.001 0.001 0.001"/>
+      </geometry>
+      <material name="black" />
+    </visual>
+  </link>
+<joint name="rear_cover_link_joint" type="fixed">
+  <origin xyz="0 0 0" rpy="0 0 0" />
+  <parent link="chassis_link"/>
+  <child link="rear_cover_link" />
+</joint>
+  <link name="rear_cover_link">
+    <visual>
+      <origin xyz="0 0 0" rpy=" 0 0 ${PI}" />
+      <geometry>
+        <mesh filename="package://ridgeback_description/meshes/end-cover.stl"  scale="0.001 0.001 0.001"/>
+      </geometry>
+      <material name="black" />
+    </visual>
+  </link>
+<joint name="top_link_joint" type="fixed">
+  <origin xyz="0 0 0" rpy="0 0 0" />
+  <parent link="chassis_link"/>
+  <child link="top_link" />
+</joint>
+  <link name="top_link">
+    <visual>
+      <origin xyz="${-chassis_length/2} ${-chassis_width/2} ${top_offset}" rpy=" ${PI/2} 0 ${PI/2}" />
+      <geometry>
+        <mesh filename="package://ridgeback_description/meshes/top.stl" />
+      </geometry>
+      <material name="black" />
+    </visual>
+  </link>
+<joint name="axle_joint" type="fixed">
+  <origin xyz="0 0 0" rpy="0 0 0" />
+  <parent link="chassis_link"/>
+  <child link="axle_link" />
+</joint>
+  <link name="axle_link">
+    <visual>
+      <origin xyz="0 0 0" rpy="0 0 0" />
+      <geometry>
+        <mesh filename="package://ridgeback_description/meshes/axle.stl" />
+      </geometry>
+      <material name="black" />
+    </visual>
   </link>
   <!-- TODO: Make this internal_imu_link or something, and use a mixed-in xacro

Commit message: Removed HW Interface for passive joint.

File: ridgeback_description/urdf/ridgeback.urdf.xacro (robot description, xacro)
@@ -96,7 +96,5 @@
   <transmission name="${prefix}_rocker_trans">
     <type>transmission_interface/SimpleTransmission</type>
-    <joint name="${prefix}_rocker">
-      <hardwareInterface>VelocityJointInterface</hardwareInterface>
-    </joint>
+    <joint name="${prefix}_rocker" />
     <actuator name="${prefix}_actuator">
       <mechanicalReduction>1</mechanicalReduction>

Commit message: Updated meshes and URDF.

File: ridgeback_description/urdf/ridgeback.urdf.xacro (robot description, xacro)
@@ -10,9 +10,8 @@
   <xacro:property name="chassis_width" value="0.787" />
   <xacro:property name="chassis_height" value="0.216" />
-  <xacro:property name="cover_offset" value="0.240" />
-  <xacro:property name="top_offset" value="0.05" />
-  <!-- Need to verify values above -->
+  <xacro:property name="axle_offset" value="0.0500" />
+  <xacro:property name="rocker_offset" value="0.301525" />
+  <xacro:property name="rocker_width" value="0.568" />
   <xacro:property name="dummy_inertia" value="1e-09"/>
-  <xacro:property name="mount_spacing" value="0.120" />
   <material name="dark_grey"><color rgba="0.2 0.2 0.2 1.0" /></material>
   <material name="light_grey"><color rgba="0.4 0.4 0.4 1.0" /></material>
@@ -71,8 +70,8 @@
     </transmission>
   </xacro:macro>
-<xacro:macro name="rocker" params="prefix joint_type wheel_location *joint_limits">
+<xacro:macro name="rocker" params="prefix joint_type location *joint_limits">
   <link name="${prefix}_rocker_link">
     <visual>
-      <origin xyz="0 0 0" rpy="0 0 0"/>
+      <origin xyz="0 0 0" rpy="${PI/2} 0 ${PI/2}" />
       <geometry>
         <mesh filename="package://ridgeback_description/meshes/rocker.stl"/>
@@ -90,5 +89,5 @@
     <parent link="axle_link"/>
     <child link="${prefix}_rocker_link" />
-    <origin xyz="0 0 0" rpy="0 0 0" />
+    <origin xyz="${location*rocker_offset} 0 0" rpy="0 0 0" />
     <axis xyz="1 0 0" />
     <xacro:insert_block name="joint_limits" />
@@ -102,14 +101,14 @@
   </transmission>
   <xacro:wheel prefix="${prefix}" side="left" y_friction="-0.707107">
-    <origin xyz="${wheel_location*wheelbase/2} ${track/2} ${wheel_vertical_offset}" rpy="0 0 0" />
+    <origin xyz="0 ${-rocker_width/2 - wheel_width/2} 0" rpy="0 0 0" />
   </xacro:wheel>
   <xacro:wheel prefix="${prefix}" side="right" y_friction="0.707107">
-    <origin xyz="${wheel_location*wheelbase/2} ${-track/2} ${wheel_vertical_offset}" rpy="0 0 0" />
+    <origin xyz="0 ${rocker_width/2 + wheel_width/2} 0" rpy="0 0 0" />
   </xacro:wheel>
 </xacro:macro>
-<xacro:rocker prefix="front" joint_type="revolute" wheel_location="1" >
+<xacro:rocker prefix="front" joint_type="revolute" location="1" >
   <limit lower="-0.2" upper="0.2" effort="0" velocity="0" />
 </xacro:rocker>
-<xacro:rocker prefix="rear" joint_type="fixed" wheel_location="-1" >
+<xacro:rocker prefix="rear" joint_type="fixed" location="-1" >
   <limit effort="0" velocity="0" />
 </xacro:rocker>
@@ -122,5 +121,5 @@
   <link name="chassis_link">
     <visual>
-      <origin xyz="0 0 0" rpy=" 0 0 0" />
+      <origin xyz="0 0 0" rpy=" ${PI/2} 0 ${PI/2}" />
       <geometry>
         <mesh filename="package://ridgeback_description/meshes/body.stl"/>
@@ -150,7 +149,7 @@
   <link name="front_cover_link">
     <visual>
-      <origin xyz="${cover_offset} ${-chassis_width/2} 0" rpy=" 0 0 0" />
-      <geometry>
-        <mesh filename="package://ridgeback_description/meshes/end-cover.stl"  scale="0.001 0.001 0.001"/>
+      <origin xyz="0 0 0" rpy=" ${PI/2} 0 ${PI/2}"  />
+      <geometry>
+        <mesh filename="package://ridgeback_description/meshes/end-cover.stl" />
       </geometry>
       <material name="black" />
@@ -164,7 +163,7 @@
   <link name="rear_cover_link">
     <visual>
-      <origin xyz="0 0 0" rpy=" 0 0 ${PI}" />
-      <geometry>
-        <mesh filename="package://ridgeback_description/meshes/end-cover.stl"  scale="0.001 0.001 0.001"/>
+      <origin xyz="0 0 0" rpy=" ${PI/2} 0 ${-PI/2}"  />
+      <geometry>
+        <mesh filename="package://ridgeback_description/meshes/end-cover.stl" />
       </geometry>
       <material name="black" />
@@ -178,5 +177,5 @@
   <link name="top_link">
     <visual>
-      <origin xyz="${-chassis_length/2} ${-chassis_width/2} ${top_offset}" rpy=" ${PI/2} 0 ${PI/2}" />
+      <origin xyz="${-chassis_length/2} ${-chassis_width/2} 0" rpy=" ${PI/2} 0 ${PI/2}" />
       <geometry>
         <mesh filename="package://ridgeback_description/meshes/top.stl" />
@@ -186,5 +185,5 @@
   </link>
 <joint name="axle_joint" type="fixed">
-  <origin xyz="0 0 0" rpy="0 0 0" />
+  <origin xyz="0 0 ${axle_offset}" rpy="0 0 0" />
   <parent link="chassis_link"/>
   <child link="axle_link" />
@@ -192,5 +191,5 @@
   <link name="axle_link">
     <visual>
-      <origin xyz="0 0 0" rpy="0 0 0" />
+      <origin xyz="0 0 0" rpy="0 ${PI/2} 0" />
       <geometry>
         <mesh filename="package://ridgeback_description/meshes/axle.stl" />

Commit message: Swapped front and rear covers to set to correct location.

File: ridgeback_description/urdf/ridgeback.urdf.xacro (robot description, xacro)
@@ -108,5 +108,5 @@
 </xacro:macro>
 <xacro:rocker prefix="front" joint_type="revolute" location="1" >
-  <limit lower="-0.2" upper="0.2" effort="0" velocity="0" />
+  <limit lower="-0.08726" upper="0.08726" effort="0" velocity="0" />
 </xacro:rocker>
 <xacro:rocker prefix="rear" joint_type="fixed" location="-1" >
@@ -149,5 +149,5 @@
   <link name="front_cover_link">
     <visual>
-      <origin xyz="0 0 0" rpy=" ${PI/2} 0 ${PI/2}"  />
+      <origin xyz="0 0 0" rpy=" ${PI/2} 0 ${-PI/2}"  />
       <geometry>
         <mesh filename="package://ridgeback_description/meshes/end-cover.stl" />
@@ -163,5 +163,5 @@
   <link name="rear_cover_link">
     <visual>
-      <origin xyz="0 0 0" rpy=" ${PI/2} 0 ${-PI/2}"  />
+      <origin xyz="0 0 0" rpy=" ${PI/2} 0 ${PI/2}"  />
       <geometry>
         <mesh filename="package://ridgeback_description/meshes/end-cover.stl" />

Commit message: Fixed collision box.

File: ridgeback_description/urdf/ridgeback.urdf.xacro (robot description, xacro)
@@ -7,5 +7,5 @@
   <xacro:property name="wheel_radius" value="0.0759" />
   <xacro:property name="wheel_width" value="0.0471" />
-  <xacro:property name="chassis_length" value="0.927" />
+  <xacro:property name="chassis_length" value="0.935" />
   <xacro:property name="chassis_width" value="0.787" />
   <xacro:property name="chassis_height" value="0.216" />
@@ -128,5 +128,5 @@
     </visual>
     <collision>
-      <origin xyz="0 0 0"/>
+      <origin xyz="0 0  ${chassis_height/2}"/>
       <geometry>
         <box size="${chassis_length} ${chassis_width} ${chassis_height}"/>

Commit message: Removed collision tag from rockers.

File: ridgeback_description/urdf/ridgeback.urdf.xacro (robot description, xacro)
@@ -79,10 +79,4 @@
       <material name="black" />
     </visual>
-    <collision>
-      <origin xyz="0 0 0" rpy="0 0 0"/>
-      <geometry>
-        <box size="${wheelbase} ${track} 0"/>
-      </geometry>
-    </collision>
   </link>
   <joint name="${prefix}_rocker" type="${joint_type}">
