Commit message: Description cleanup for simulation
Fixed a few bad references and inertia/materials issues,
as well as just general indentation cleanup. Inertia/mass
info is still just dummy for now, will have to be cleaned
up later.

File: ridgeback_description/urdf/ridgeback.urdf.xacro (robot description, xacro)
@@ -34,24 +34,12 @@
       </collision>
       <inertial>
-        <origin xyz="-0.0001 0 -0.00001" rpy="0 0 0"/>
+        <origin xyz="0 0 0" rpy="0 0 0"/>
         <mass value="0.477"/>
         <inertia
-          ixx="0.0024" ixy="0" ixz="0"
-          iyy="0.0013" iyz="0"
+          ixx="0.0013" ixy="0" ixz="0"
+          iyy="0.0024" iyz="0"
           izz="0.0013"/>
       </inertial>
     </link>
-    <gazebo reference="${prefix}_${side}_wheel_link">
-      <material>Gazebo/DarkGrey</material>
-      <friction>
-        <ode>
-          <fdir1>0.707107 ${y_friction} 0.000000</fdir1>
-          <mu1>0.0001</mu1>
-          <mu2>1000</mu2>
-          <slip1>1000</slip1>
-          <slip2>0.0001</slip2>
-        </ode>
-      </friction>
-    </gazebo>
     <joint name="${prefix}_${side}_wheel" type="continuous">
       <parent link="${prefix}_rocker_link"/>
@@ -62,5 +50,5 @@
     <transmission name="${prefix}_wheel_trans">
       <type>transmission_interface/SimpleTransmission</type>
-      <joint name="${prefix}_wheel">
+      <joint name="${prefix}_${side}_wheel">
         <hardwareInterface>VelocityJointInterface</hardwareInterface>
       </joint>
@@ -70,41 +58,42 @@
     </transmission>
   </xacro:macro>
-<xacro:macro name="rocker" params="prefix joint_type location *joint_limits">
-  <link name="${prefix}_rocker_link">
-    <visual>
-      <origin xyz="0 0 0" rpy="${PI/2} 0 ${PI/2}" />
-      <geometry>
-        <mesh filename="package://ridgeback_description/meshes/rocker.stl"/>
-      </geometry>
-      <material name="black" />
-    </visual>
-  </link>
-  <joint name="${prefix}_rocker" type="${joint_type}">
-    <parent link="axle_link"/>
-    <child link="${prefix}_rocker_link" />
-    <origin xyz="${location*rocker_offset} 0 0" rpy="0 0 0" />
-    <axis xyz="1 0 0" />
-    <xacro:insert_block name="joint_limits" />
-  </joint>
-  <transmission name="${prefix}_rocker_trans">
-    <type>transmission_interface/SimpleTransmission</type>
-    <joint name="${prefix}_rocker" />
-    <actuator name="${prefix}_actuator">
-      <mechanicalReduction>1</mechanicalReduction>
-    </actuator>
-  </transmission>
-  <xacro:wheel prefix="${prefix}" side="left" y_friction="-0.707107">
-    <origin xyz="0 ${-rocker_width/2 - wheel_width/2} 0" rpy="0 0 0" />
-  </xacro:wheel>
-  <xacro:wheel prefix="${prefix}" side="right" y_friction="0.707107">
-    <origin xyz="0 ${rocker_width/2 + wheel_width/2} 0" rpy="0 0 0" />
-  </xacro:wheel>
-</xacro:macro>
-<xacro:rocker prefix="front" joint_type="revolute" location="1" >
-  <limit lower="-0.08726" upper="0.08726" effort="0" velocity="0" />
-</xacro:rocker>
-<xacro:rocker prefix="rear" joint_type="fixed" location="-1" >
-  <limit effort="0" velocity="0" />
-</xacro:rocker>
+  <xacro:macro name="rocker" params="prefix joint_type location *joint_limits">
+    <link name="${prefix}_rocker_link">
+      <visual>
+        <origin xyz="0 0 0" rpy="${PI/2} 0 ${PI/2}" />
+        <geometry>
+          <mesh filename="package://ridgeback_description/meshes/rocker.stl"/>
+        </geometry>
+        <material name="black" />
+      </visual>
+      <inertial>
+        <origin xyz="0 0 0" rpy="0 0 0"/>
+        <mass value="3"/>
+        <inertia
+          ixx="0.001" ixy="0" ixz="0"
+          iyy="0.001" iyz="0"
+          izz="0.001"/>
+      </inertial>
+    </link>
+    <joint name="${prefix}_rocker" type="${joint_type}">
+      <parent link="axle_link"/>
+      <child link="${prefix}_rocker_link" />
+      <origin xyz="${location*rocker_offset} 0 0" rpy="0 0 0" />
+      <axis xyz="1 0 0" />
+      <xacro:insert_block name="joint_limits" />
+    </joint>
+    <xacro:wheel prefix="${prefix}" side="left" y_friction="-0.707107">
+      <origin xyz="0 ${-rocker_width/2 - wheel_width/2} 0" rpy="0 0 0" />
+    </xacro:wheel>
+    <xacro:wheel prefix="${prefix}" side="right" y_friction="0.707107">
+      <origin xyz="0 ${rocker_width/2 + wheel_width/2} 0" rpy="0 0 0" />
+    </xacro:wheel>
+  </xacro:macro>
+  <xacro:rocker prefix="front" joint_type="revolute" location="1" >
+    <limit lower="-0.08726" upper="0.08726" effort="0" velocity="0" />
+  </xacro:rocker>
+  <xacro:rocker prefix="rear" joint_type="fixed" location="-1" >
+    <limit effort="0" velocity="0" />
+  </xacro:rocker>
   <link name="base_link"></link>
   <joint name="base_link_joint" type="fixed">
@@ -128,17 +117,17 @@
     </collision>
     <inertial>
-      <origin xyz="0.012  0.002 0.067" rpy="0 0 0"/>
-      <mass value="16.523"/>
+      <origin xyz="0.012 0.002 0.067" rpy="0 0 0"/>
+      <mass value="50"/>
       <inertia
-        ixx="0.3136" ixy="-0.0008" ixz="0.0164"
-        iyy="0.3922" iyz="-0.0009"
-        izz="0.4485"/>
+        ixx="1.3136" ixy="0.0" ixz="0.0"
+        iyy="1.3922" iyz="0.0"
+        izz="2.0"/>
     </inertial>
   </link>
-<joint name="front_cover_link_joint" type="fixed">
-  <origin xyz="0 0 0" rpy="0 0 0" />
-  <parent link="chassis_link"/>
-  <child link="front_cover_link" />
-</joint>
+  <joint name="front_cover_link_joint" type="fixed">
+    <origin xyz="0 0 0" rpy="0 0 0" />
+    <parent link="chassis_link"/>
+    <child link="front_cover_link" />
+  </joint>
   <link name="front_cover_link">
     <visual>
@@ -150,9 +139,9 @@
     </visual>
   </link>
-<joint name="rear_cover_link_joint" type="fixed">
-  <origin xyz="0 0 0" rpy="0 0 0" />
-  <parent link="chassis_link"/>
-  <child link="rear_cover_link" />
-</joint>
+  <joint name="rear_cover_link_joint" type="fixed">
+    <origin xyz="0 0 0" rpy="0 0 0" />
+    <parent link="chassis_link"/>
+    <child link="rear_cover_link" />
+  </joint>
   <link name="rear_cover_link">
     <visual>
@@ -164,9 +153,9 @@
     </visual>
   </link>
-<joint name="top_link_joint" type="fixed">
-  <origin xyz="0 0 0" rpy="0 0 0" />
-  <parent link="chassis_link"/>
-  <child link="top_link" />
-</joint>
+  <joint name="top_link_joint" type="fixed">
+    <origin xyz="0 0 0" rpy="0 0 0" />
+    <parent link="chassis_link"/>
+    <child link="top_link" />
+  </joint>
   <link name="top_link">
     <visual>
@@ -178,9 +167,9 @@
     </visual>
   </link>
-<joint name="axle_joint" type="fixed">
-  <origin xyz="0 0 ${axle_offset}" rpy="0 0 0" />
-  <parent link="chassis_link"/>
-  <child link="axle_link" />
-</joint>
+  <joint name="axle_joint" type="fixed">
+    <origin xyz="0 0 ${axle_offset}" rpy="0 0 0" />
+    <parent link="chassis_link"/>
+    <child link="axle_link" />
+  </joint>
   <link name="axle_link">
     <visual>
@@ -208,5 +197,5 @@
   </joint>
   <!-- Bring in simulation data for Gazebo. -->
-  <!--<xacro:include filename="ridgeback.gazebo" />-->
+  <xacro:include filename="ridgeback.gazebo" />
   <!-- Optional standard accessories, including their simulation data. The rendering
        of these into the final description is controlled by optenv variables, which

Commit message: Add simulator plugins.

File: ridgeback_description/urdf/ridgeback.urdf.xacro (robot description, xacro)
@@ -18,5 +18,5 @@
   <material name="yellow"><color rgba="0.8 0.8 0.0 1.0" /></material>
   <material name="black"><color rgba="0.15 0.15 0.15 1.0" /></material>
-  <xacro:macro name="wheel" params="prefix side y_friction *joint_pose">
+  <xacro:macro name="wheel" params="prefix side *joint_pose">
     <link name="${prefix}_${side}_wheel_link">
       <visual>
@@ -83,9 +83,9 @@
       <xacro:insert_block name="joint_limits" />
     </joint>
-    <xacro:wheel prefix="${prefix}" side="left" y_friction="-0.707107">
-      <origin xyz="0 ${-rocker_width/2 - wheel_width/2} 0" rpy="0 0 0" />
+    <xacro:wheel prefix="${prefix}" side="left">
+      <origin xyz="0 ${rocker_width/2 + wheel_width/2} 0" rpy="0 0 0" />
     </xacro:wheel>
-    <xacro:wheel prefix="${prefix}" side="right" y_friction="0.707107">
-      <origin xyz="0 ${rocker_width/2 + wheel_width/2} 0" rpy="0 0 0" />
+    <xacro:wheel prefix="${prefix}" side="right">
+      <origin xyz="0 ${-(rocker_width/2 + wheel_width/2)} 0" rpy="0 0 0" />
     </xacro:wheel>
   </xacro:macro>

Commit message: Fixed wheel positions in urdf.

File: ridgeback_description/urdf/ridgeback.urdf.xacro (robot description, xacro)
@@ -84,8 +84,8 @@
     </joint>
     <xacro:wheel prefix="${prefix}" side="left" y_friction="-0.707107">
-      <origin xyz="0 ${-rocker_width/2 - wheel_width/2} 0" rpy="0 0 0" />
+      <origin xyz="0 ${rocker_width/2 + wheel_width/2} 0" rpy="0 0 0" />
     </xacro:wheel>
     <xacro:wheel prefix="${prefix}" side="right" y_friction="0.707107">
-      <origin xyz="0 ${rocker_width/2 + wheel_width/2} 0" rpy="0 0 0" />
+      <origin xyz="0 ${-rocker_width/2 - wheel_width/2} 0" rpy="0 0 0" />
     </xacro:wheel>
   </xacro:macro>

Commit message: Updated URDF for physical changes.

File: ridgeback_description/urdf/ridgeback.urdf.xacro (robot description, xacro)
@@ -2,16 +2,13 @@
 <robot name="ridgeback" xmlns:xacro="http://www.ros.org/wiki/xacro">
   <xacro:property name="PI" value="3.1415926535897931" />
-  <xacro:property name="wheelbase" value="0.610" />
-  <xacro:property name="track" value="0.622" />
-  <xacro:property name="wheel_vertical_offset" value="0.05" />
   <xacro:property name="wheel_radius" value="0.0759" />
-  <xacro:property name="wheel_width" value="0.0471" />
-  <xacro:property name="chassis_length" value="0.935" />
-  <xacro:property name="chassis_width" value="0.787" />
+  <xacro:property name="wheel_width" value="0.0790" />
+  <xacro:property name="chassis_length" value="0.960" />
+  <xacro:property name="chassis_width" value="0.793" />
   <xacro:property name="chassis_height" value="0.216" />
   <xacro:property name="deck_height" value="0.280" />
   <xacro:property name="axle_offset" value="0.0500" />
-  <xacro:property name="rocker_offset" value="0.301525" />
-  <xacro:property name="rocker_width" value="0.568" />
+  <xacro:property name="rocker_offset" value="0.319" />
+  <xacro:property name="rocker_width" value="0.472" />
   <xacro:property name="dummy_inertia" value="1e-09"/>
   <material name="dark_grey"><color rgba="0.2 0.2 0.2 1.0" /></material>

Commit message: Fixed IMU offset.

File: ridgeback_description/urdf/ridgeback.urdf.xacro (robot description, xacro)
@@ -11,4 +11,7 @@
   <xacro:property name="rocker_offset" value="0.319" />
   <xacro:property name="rocker_width" value="0.472" />
+  <xacro:property name="imu_offset_x" value="0.2085" />
+  <xacro:property name="imu_offset_y" value="-0.2902" />
+  <xacro:property name="imu_offset_z" value="0.1681" />
   <xacro:property name="dummy_inertia" value="1e-09"/>
   <material name="dark_grey"><color rgba="0.2 0.2 0.2 1.0" /></material>
@@ -189,4 +192,5 @@
     <parent link="chassis_link" />
     <child link="imu_link" />
+    <origin xyz="${imu_offset_x} ${imu_offset_y} ${imu_offset_z}" rpy="0 0 0"/>
   </joint>
   <link name="mid_mount" />

Commit message: Updated material properties for Ridgeback.

File: ridgeback_description/urdf/ridgeback.urdf.xacro (robot description, xacro)
@@ -36,9 +36,9 @@
       <inertial>
         <origin xyz="0 0 0" rpy="0 0 0"/>
-        <mass value="0.477"/>
+        <mass value="2.3"/>
         <inertia
-          ixx="0.0013" ixy="0" ixz="0"
-          iyy="0.0024" iyz="0"
-          izz="0.0013"/>
+          ixx="3.3212e-3" ixy="0" ixz="0"
+          iyy="6.6424e-3" iyz="0"
+          izz="3.3212e-3"/>
       </inertial>
     </link>
@@ -69,10 +69,10 @@
       </visual>
       <inertial>
-        <origin xyz="0 0 0" rpy="0 0 0"/>
-        <mass value="3"/>
+        <origin xyz="0 0 0" rpy="${PI/2} 0 ${PI/2}"/>
+        <mass value="10.267"/>
         <inertia
-          ixx="0.001" ixy="0" ixz="0"
-          iyy="0.001" iyz="0"
-          izz="0.001"/>
+          ixx="0.0288" ixy="2.20484e-6" ixz="-1.3145e-5"
+          iyy="0.4324" iyz="1.8944e-3"
+          izz="0.4130"/>
       </inertial>
     </link>
@@ -105,5 +105,5 @@
   <link name="chassis_link">
     <visual>
-      <origin xyz="0 0 0" rpy=" ${PI/2} 0 ${PI/2}" />
+      <origin xyz="0 0 0" rpy="${PI/2} 0 ${PI/2}" />
       <geometry>
         <mesh filename="package://ridgeback_description/meshes/body.stl"/>
@@ -112,16 +112,16 @@
     </visual>
     <collision>
-      <origin xyz="0 0 ${chassis_height/2}"/>
-      <geometry>
-        <box size="${chassis_length} ${chassis_width} ${chassis_height}"/>
+      <origin xyz="0 0 ${deck_height/2}"/>
+      <geometry>
+        <box size="${chassis_length} ${chassis_width} ${deck_height}"/>
       </geometry>
     </collision>
     <inertial>
-      <origin xyz="0.012 0.002 0.067" rpy="0 0 0"/>
-      <mass value="50"/>
+      <origin xyz="0.012 0.002 0.067" rpy="${PI/2} 0 ${PI/2}"/>
+      <mass value="165.304"/>
       <inertia
-        ixx="1.3136" ixy="0.0" ixz="0.0"
-        iyy="1.3922" iyz="0.0"
-        izz="2.0"/>
+        ixx="4.4744" ixy="0.03098" ixz="0.003647"
+        iyy="7.1624" iyz="0.1228"
+        izz="4.6155"/>
     </inertial>
   </link>

Commit message: Reverted dimensions of chassis collision mesh to allow laser rays out.

File: ridgeback_description/urdf/ridgeback.urdf.xacro (robot description, xacro)
@@ -112,7 +112,7 @@
     </visual>
     <collision>
-      <origin xyz="0 0 ${deck_height/2}"/>
-      <geometry>
-        <box size="${chassis_length} ${chassis_width} ${deck_height}"/>
+      <origin xyz="0 0 ${chassis_height/2}"/>
+      <geometry>
+        <box size="${chassis_length} ${chassis_width} ${chassis_height}"/>
       </geometry>
     </collision>

Commit message: Updated the visual meshes to make them lighter and prettier.  More accurate collision mesh made for tight areas

File: ridgeback_description/urdf/ridgeback.urdf.xacro (robot description, xacro)
@@ -17,4 +17,6 @@
   <material name="dark_grey"><color rgba="0.2 0.2 0.2 1.0" /></material>
   <material name="light_grey"><color rgba="0.4 0.4 0.4 1.0" /></material>
+  <material name="red"><color rgba="0.8 0.0 0.0 1.0" /></material>
+  <material name="white"><color rgba="0.9 0.9 0.9 1.0" /></material>
   <material name="yellow"><color rgba="0.8 0.8 0.0 1.0" /></material>
   <material name="black"><color rgba="0.15 0.15 0.15 1.0" /></material>
@@ -105,5 +107,5 @@
   <link name="chassis_link">
     <visual>
-      <origin xyz="0 0 0" rpy="${PI/2} 0 ${PI/2}" />
+      <origin xyz="0 0 0" rpy="0 0 0" />
       <geometry>
         <mesh filename="package://ridgeback_description/meshes/body.stl"/>
@@ -112,7 +114,7 @@
     </visual>
     <collision>
-      <origin xyz="0 0 ${chassis_height/2}"/>
-      <geometry>
-        <box size="${chassis_length} ${chassis_width} ${chassis_height}"/>
+      <origin xyz="0 0 0"/>
+      <geometry>
+        <mesh filename="package://ridgeback_description/meshes/body-collision.stl"/>
       </geometry>
     </collision>
@@ -126,4 +128,32 @@
     </inertial>
   </link>
+  <joint name="right_side_cover_link_joint" type="fixed">
+    <origin xyz="0 0 0" rpy="0 0 0" />
+    <parent link="chassis_link"/>
+    <child link="right_side_cover_link" />
+  </joint>
+  <joint name="left_side_cover_link_joint" type="fixed">
+    <origin xyz="0 0 0" rpy="0 0 0" />
+    <parent link="chassis_link"/>
+    <child link="left_side_cover_link" />
+  </joint>
+  <link name="left_side_cover_link">
+    <visual>
+      <origin xyz="0 0 0" rpy="0 0 ${PI}" />
+      <geometry>
+        <mesh filename="package://ridgeback_description/meshes/side-cover.stl"/>
+      </geometry>
+      <material name="yellow" />
+    </visual>
+  </link>
+  <link name="right_side_cover_link">
+    <visual>
+      <origin xyz="0 0 0" rpy="0 0 0" />
+      <geometry>
+        <mesh filename="package://ridgeback_description/meshes/side-cover.stl"/>
+      </geometry>
+      <material name="yellow" />
+    </visual>
+  </link>
   <joint name="front_cover_link_joint" type="fixed">
     <origin xyz="0 0 0" rpy="0 0 0" />
@@ -133,5 +163,5 @@
   <link name="front_cover_link">
     <visual>
-      <origin xyz="0 0 0" rpy=" ${PI/2} 0 ${-PI/2}"  />
+      <origin xyz="0 0 0" rpy="0 0 0" />
       <geometry>
         <mesh filename="package://ridgeback_description/meshes/end-cover.stl" />
@@ -147,5 +177,5 @@
   <link name="rear_cover_link">
     <visual>
-      <origin xyz="0 0 0" rpy=" ${PI/2} 0 ${PI/2}"  />
+      <origin xyz="0 0 0" rpy="0 0 ${PI}" />
       <geometry>
         <mesh filename="package://ridgeback_description/meshes/end-cover.stl" />
@@ -154,4 +184,32 @@
     </visual>
   </link>
+  <joint name="front_lights_link_joint" type="fixed">
+    <origin xyz="0 0 0" rpy="0 0 0" />
+    <parent link="chassis_link"/>
+    <child link="front_lights_link" />
+  </joint>
+  <joint name="rear_lights_link_joint" type="fixed">
+    <origin xyz="0 0 0" rpy="0 0 0" />
+    <parent link="chassis_link"/>
+    <child link="rear_lights_link" />
+  </joint>
+  <link name="front_lights_link">
+    <visual>
+      <origin xyz="0 0 0" rpy="0 0 0" />
+      <geometry>
+        <mesh filename="package://ridgeback_description/meshes/lights.stl" />
+      </geometry>
+      <material name="white" />
+    </visual>
+  </link>
+  <link name="rear_lights_link">
+    <visual>
+      <origin xyz="0 0 0" rpy="0 0 ${PI}" />
+      <geometry>
+        <mesh filename="package://ridgeback_description/meshes/lights.stl" />
+      </geometry>
+      <material name="red" />
+    </visual>
+  </link>
   <joint name="top_link_joint" type="fixed">
     <origin xyz="0 0 0" rpy="0 0 0" />
@@ -161,5 +219,5 @@
   <link name="top_link">
     <visual>
-      <origin xyz="${-chassis_length/2} ${-chassis_width/2} 0" rpy=" ${PI/2} 0 ${PI/2}" />
+      <origin xyz="0 0 0" rpy="0 0 0" />
       <geometry>
         <mesh filename="package://ridgeback_description/meshes/top.stl" />
@@ -167,4 +225,10 @@
       <material name="black" />
     </visual>
+    <collision>
+      <origin xyz="0 0 0" rpy="0 0 0" />
+      <geometry>
+        <mesh filename="package://ridgeback_description/meshes/top.stl"/>
+      </geometry>
+    </collision>
   </link>
   <joint name="axle_joint" type="fixed">

Commit message: Initial commit of adding a customizable riser height to the URDF

File: ridgeback_description/urdf/ridgeback.urdf.xacro (robot description, xacro)
@@ -8,4 +8,5 @@
   <xacro:property name="chassis_height" value="0.216" />
   <xacro:property name="deck_height" value="0.280" />
+  <xacro:property name="riser_height" value="$(optenv RIDGEBACK_RISER_HEIGHT 0.055)" />
   <xacro:property name="axle_offset" value="0.0500" />
   <xacro:property name="rocker_offset" value="0.319" />
@@ -128,4 +129,24 @@
     </inertial>
   </link>
+  <link name="riser_link">
+    <visual>
+      <origin xyz="0 0 ${riser_height/2}" rpy="0 0 ${pi/4}" />
+      <geometry>
+        <box size="0.493 0.493 ${riser_height}" />
+      </geometry>
+      <material name="black" />
+    </visual>
+    <collision>
+      <origin xyz="0 0 ${riser_height/2}" rpy="0 0 ${pi/4}" />
+      <geometry>
+        <box size="0.493 0.493 ${riser_height}" />
+      </geometry>
+    </collision>
+  </link>
+  <joint name="riser_link_joint" type="fixed">
+    <origin xyz="0 0 0.225" rpy="0 0 0" />
+    <parent link="chassis_link" />
+    <child link="riser_link" />
+  </joint>
   <joint name="right_side_cover_link_joint" type="fixed">
     <origin xyz="0 0 0" rpy="0 0 0" />
@@ -209,10 +230,10 @@
         <mesh filename="package://ridgeback_description/meshes/lights.stl" />
       </geometry>
-      <material name="red" />
+      <material name="black" />
     </visual>
   </link>
   <joint name="top_link_joint" type="fixed">
-    <origin xyz="0 0 0" rpy="0 0 0" />
-    <parent link="chassis_link"/>
+    <origin xyz="0 0 ${riser_height-deck_height}" rpy="0 0 0" />
+    <parent link="riser_link"/>
     <child link="top_link" />
   </joint>
@@ -260,7 +281,7 @@
   <link name="mid_mount" />
   <joint name="mid_mount_joint" type="fixed">
-    <parent link="base_link" />
+    <parent link="riser_link" />
     <child link="mid_mount" />
-    <origin xyz="0 0 ${deck_height}" rpy="0 0 0"/>
+    <origin xyz="0 0 ${riser_height}" rpy="0 0 0"/>
   </joint>
   <!-- Bring in simulation data for Gazebo. -->

Commit message: Take the thickness of the deck into consideration so that the riser link has the correct origin and the top link sits atop it correctly. Change the riser colour to light grey to match the unfinished aluminium extrusion used for this component

File: ridgeback_description/urdf/ridgeback.urdf.xacro (robot description, xacro)
@@ -8,4 +8,5 @@
   <xacro:property name="chassis_height" value="0.216" />
   <xacro:property name="deck_height" value="0.280" />
+  <xacro:property name="deck_thickness" value="0.005" />
   <xacro:property name="riser_height" value="$(optenv RIDGEBACK_RISER_HEIGHT 0.055)" />
   <xacro:property name="axle_offset" value="0.0500" />
@@ -135,5 +136,5 @@
         <box size="0.493 0.493 ${riser_height}" />
       </geometry>
-      <material name="black" />
+      <material name="light_grey" />
     </visual>
     <collision>
@@ -145,5 +146,5 @@
   </link>
   <joint name="riser_link_joint" type="fixed">
-    <origin xyz="0 0 0.225" rpy="0 0 0" />
+    <origin xyz="0 0 ${0.225 - deck_thickness}" rpy="0 0 0" />
     <parent link="chassis_link" />
     <child link="riser_link" />
@@ -234,5 +235,5 @@
   </link>
   <joint name="top_link_joint" type="fixed">
-    <origin xyz="0 0 ${riser_height-deck_height}" rpy="0 0 0" />
+    <origin xyz="0 0 ${riser_height-deck_height+deck_thickness}" rpy="0 0 0" />
     <parent link="riser_link"/>
     <child link="top_link" />
@@ -283,5 +284,5 @@
     <parent link="riser_link" />
     <child link="mid_mount" />
-    <origin xyz="0 0 ${riser_height}" rpy="0 0 0"/>
+    <origin xyz="0 0 ${riser_height + deck_thickness}" rpy="0 0 0"/>
   </joint>
   <!-- Bring in simulation data for Gazebo. -->
