Commit message: Made rear laser optional and removed un-needed files.

File: ridgeback_description/urdf/accessories.urdf.xacro (robot description, xacro)
@@ -9,31 +9,10 @@
     ridgeback_base/launch/base.launch
   -->
-  <!-- Macros to generate standoffs for offset payload mounting. -->
-  <xacro:include filename="accessories/standoffs.urdf.xacro" />
-  <!-- This optional plate mounts both the upgraded GPS and the Velodyne 3D LIDAR. -->
-  <xacro:include filename="accessories/bridge_plate.urdf.xacro" />
-  <!-- If enabled, generate the LASER payload (by default, a SICK LMS111). -->
-  <xacro:include filename="accessories/sick_lms1xx.urdf.xacro" />
-  <xacro:if value="$(optenv JACKAL_LASER 0)">
-    <sick_lms1xx_mount prefix="$(optenv JACKAL_LASER_MOUNT front)"
-                       topic="$(optenv JACKAL_LASER_TOPIC scan)" />
-    <joint name="$front_laser_mount_joint" type="fixed">
-      <origin xyz="$(optenv JACKAL_LASER_OFFSET 0 0 0)"
-              rpy="$(optenv JACKAL_LASER_RPY 0 0 0)" />
-      <parent link="$(optenv JACKAL_LASER_MOUNT front)_mount" />
-      <child link="$(optenv JACKAL_LASER_MOUNT front)_laser_mount" />
-    </joint>
-  </xacro:if>
-  <!-- If enabled, generate the upgraded Navsat payload (a Novatel Smart6). -->
-  <xacro:include filename="accessories/novatel_smart6.urdf.xacro" />
-  <xacro:if value="$(optenv JACKAL_NAVSAT 0)">
-    <bridge_plate mount="$(optenv JACKAL_NAVSAT_MOUNT rear)"
-                  height="$(optenv JACKAL_NAVSAT_HEIGHT 0.1)" />
-    <novatel_smart6 prefix="$(optenv JACKAL_NAVSAT_MOUNT rear)"/>
-    <joint name="$(optenv JACKAL_NAVSAT_MOUNT rear)_navsat_joint" type="fixed">
-      <origin xyz="0 0 0" rpy="0 0 0" />
-      <parent link="$(optenv JACKAL_NAVSAT_MOUNT rear)_bridge" />
-      <child link="$(optenv JACKAL_NAVSAT_MOUNT rear)_navsat" />
-    </joint>
+  <!-- If enabled, generate the rear LASER payload (by default, a SICK LMS111). -->
+  <xacro:include filename="accessories/sick_lms1xx_mount.urdf.xacro" />
+  <xacro:if value="$(optenv RIDGEBACK_REAR_LASER 0)">
+    <xacro:sick_lms1xx_mount prefix="$(optenv RIDGEBACK_REAR__LASER_MOUNT rear)"
+                            topic="$(optenv RIDGEBACK_REAR__LASER_TOPIC rear)"
+                            location="-1" />
   </xacro:if>
   <!--

File: ridgeback_description/urdf/accessories/sick_lms1xx_mount.urdf.xacro (robot description, xacro)
@@ -1,6 +1,5 @@
 <?xml version="1.0"?>
 <!--
-Copyright (c) 2013, Goncalo Cabrita, ISR University of Coimbra
-Copyright (c) 2014, 2015 Clearpath Robotics
+Copyright (c) 2015 Clearpath Robotics
 All rights reserved.
 Redistribution and use in source and binary forms, with or without

File: ridgeback_description/urdf/ridgeback.urdf.xacro (robot description, xacro)
@@ -198,5 +198,4 @@
   </joint>
   <xacro:sick_lms1xx_mount prefix="front" topic="front_scan" location="1" />
-  <xacro:sick_lms1xx_mount prefix="rear" topic="rear_scan" location="-1" />
   <!-- Bring in simulation data for Gazebo. -->
   <xacro:include filename="ridgeback.gazebo" />
@@ -204,5 +203,5 @@
        of these into the final description is controlled by optenv variables, which
        default each one to off.-->
-  <!--<xacro:include filename="accessories.urdf.xacro" />-->
+  <xacro:include filename="accessories.urdf.xacro" />
   <!-- Optional custom includes. -->
   <!--<xacro:include filename="$(optenv RIDGEBACK_URDF_EXTRAS empty.urdf)" />-->

Commit message: Updated to work with changes to lms1xx urdf macro.

File: ridgeback_description/urdf/accessories.urdf.xacro (robot description, xacro)
@@ -13,5 +13,5 @@
   <xacro:if value="$(optenv RIDGEBACK_FRONT_LASER 0)">
     <xacro:sick_lms1xx_mount prefix="$(optenv RIDGEBACK_FRONT_LASER_MOUNT front)"
-                            topic="$(optenv RIDGEBACK_FRONT_LASER_TOPIC scan)"
+                            topic="$(optenv RIDGEBACK_FRONT_LASER_TOPIC front/scan)"
                             location="1" />
   </xacro:if>
@@ -19,5 +19,5 @@
   <xacro:if value="$(optenv RIDGEBACK_REAR_LASER 0)">
     <xacro:sick_lms1xx_mount prefix="$(optenv RIDGEBACK_REAR__LASER_MOUNT rear)"
-                            topic="$(optenv RIDGEBACK_REAR_LASER_TOPIC scan)"
+                            topic="$(optenv RIDGEBACK_REAR_LASER_TOPIC rear/scan)"
                             location="-1" />
   </xacro:if>

File: ridgeback_description/urdf/accessories/sick_lms1xx_mount.urdf.xacro (robot description, xacro)
@@ -27,10 +27,10 @@
   <xacro:include filename="$(find lms1xx)/urdf/sick_lms1xx.urdf.xacro" />
   <xacro:macro name="sick_lms1xx_mount" params="prefix topic location">
-    <xacro:sick_lms1xx prefix="${prefix}" topic="${topic}" />
+    <xacro:sick_lms1xx frame="${prefix}_laser" topic="${topic}" />
     <joint name="${prefix}_laser_joint" type="fixed">
       <!-- This offset is from the base of the bracket to the LIDAR's focal point. -->
       <origin xyz="${location * 0.3999} 0 0.2337" rpy="0 0 ${PI/2 - (location * PI/2)}" />
       <parent link="chassis_link" />
-      <child link="${prefix}laser" />
+      <child link="${prefix}_laser" />
     </joint>
   </xacro:macro>

Commit message: Ignore ridgeback_navigation, go to planar move plugin for movement.

File: ridgeback_description/urdf/accessories.urdf.xacro (robot description, xacro)
@@ -9,5 +9,5 @@
     ridgeback_base/launch/base.launch
   -->
-  <xacro:include filename="accessories/sick_lms1xx_mount.urdf.xacro" />
+  <xacro:include filename="$(find ridgeback_description)/urdf/accessories/sick_lms1xx_mount.urdf.xacro" />
   <!-- If enabled, generate the front LASER payload (by default enabled and a SICK LMS111). -->
   <xacro:if value="$(optenv RIDGEBACK_FRONT_LASER 0)">

File: ridgeback_description/urdf/ridgeback.urdf.xacro (robot description, xacro)
@@ -10,4 +10,5 @@
   <xacro:property name="chassis_width" value="0.787" />
   <xacro:property name="chassis_height" value="0.216" />
+  <xacro:property name="deck_height" value="0.280" />
   <xacro:property name="axle_offset" value="0.0500" />
   <xacro:property name="rocker_offset" value="0.301525" />
@@ -111,5 +112,5 @@
     </visual>
     <collision>
-      <origin xyz="0 0  ${chassis_height/2}"/>
+      <origin xyz="0 0 ${chassis_height/2}"/>
       <geometry>
         <box size="${chassis_length} ${chassis_width} ${chassis_height}"/>
@@ -181,8 +182,4 @@
     </visual>
   </link>
-  <!-- TODO: Make this internal_imu_link or something, and use a mixed-in xacro
-       to supply the joint between it and imu_link. This is important so that imu_link
-       always points to the "active" IMU. When an upgrade IMU is connected, the
-       internal_imu_link should remain, but imu_link should point to the upgrade one. -->
   <link name="imu_link">
     <inertial>
@@ -196,10 +193,16 @@
     <child link="imu_link" />
   </joint>
+  <link name="mid_mount" />
+  <joint name="mid_mount_joint" type="fixed">
+    <parent link="base_link" />
+    <child link="mid_mount" />
+    <origin xyz="0 0 ${deck_height}" rpy="0 0 0"/>
+  </joint>
   <!-- Bring in simulation data for Gazebo. -->
-  <xacro:include filename="ridgeback.gazebo" />
+  <xacro:include filename="$(find ridgeback_description)/urdf/ridgeback.gazebo" />
   <!-- Optional standard accessories, including their simulation data. The rendering
        of these into the final description is controlled by optenv variables, which
        default each one to off.-->
-  <xacro:include filename="accessories.urdf.xacro" />
+  <xacro:include filename="$(find ridgeback_description)/urdf/accessories.urdf.xacro" />
   <!-- Optional custom includes. -->
   <!--<xacro:include filename="$(optenv RIDGEBACK_URDF_EXTRAS empty.urdf)" />-->

Commit message: Simulation using gazebo_ros_force_based_move.

File: ridgeback_description/urdf/accessories.urdf.xacro (robot description, xacro)
@@ -9,5 +9,5 @@
     ridgeback_base/launch/base.launch
   -->
-  <xacro:include filename="accessories/sick_lms1xx_mount.urdf.xacro" />
+  <xacro:include filename="$(find ridgeback_description)/urdf/accessories/sick_lms1xx_mount.urdf.xacro" />
   <!-- If enabled, generate the front LASER payload (by default enabled and a SICK LMS111). -->
   <xacro:if value="$(optenv RIDGEBACK_FRONT_SICK_LASER 0)">

File: ridgeback_description/urdf/ridgeback.urdf.xacro (robot description, xacro)
@@ -10,4 +10,5 @@
   <xacro:property name="chassis_width" value="0.787" />
   <xacro:property name="chassis_height" value="0.216" />
+  <xacro:property name="deck_height" value="0.280" />
   <xacro:property name="axle_offset" value="0.0500" />
   <xacro:property name="rocker_offset" value="0.301525" />
@@ -18,5 +19,5 @@
   <material name="yellow"><color rgba="0.8 0.8 0.0 1.0" /></material>
   <material name="black"><color rgba="0.15 0.15 0.15 1.0" /></material>
-  <xacro:macro name="wheel" params="prefix side y_friction *joint_pose">
+  <xacro:macro name="wheel" params="prefix side *joint_pose">
     <link name="${prefix}_${side}_wheel_link">
       <visual>
@@ -83,9 +84,9 @@
       <xacro:insert_block name="joint_limits" />
     </joint>
-    <xacro:wheel prefix="${prefix}" side="left" y_friction="-0.707107">
+    <xacro:wheel prefix="${prefix}" side="left">
       <origin xyz="0 ${rocker_width/2 + wheel_width/2} 0" rpy="0 0 0" />
     </xacro:wheel>
-    <xacro:wheel prefix="${prefix}" side="right" y_friction="0.707107">
-      <origin xyz="0 ${-rocker_width/2 - wheel_width/2} 0" rpy="0 0 0" />
+    <xacro:wheel prefix="${prefix}" side="right">
+      <origin xyz="0 ${-(rocker_width/2 + wheel_width/2)} 0" rpy="0 0 0" />
     </xacro:wheel>
   </xacro:macro>
@@ -111,5 +112,5 @@
     </visual>
     <collision>
-      <origin xyz="0 0  ${chassis_height/2}"/>
+      <origin xyz="0 0 ${chassis_height/2}"/>
       <geometry>
         <box size="${chassis_length} ${chassis_width} ${chassis_height}"/>
@@ -181,8 +182,4 @@
     </visual>
   </link>
-  <!-- TODO: Make this internal_imu_link or something, and use a mixed-in xacro
-       to supply the joint between it and imu_link. This is important so that imu_link
-       always points to the "active" IMU. When an upgrade IMU is connected, the
-       internal_imu_link should remain, but imu_link should point to the upgrade one. -->
   <link name="imu_link">
     <inertial>
@@ -196,10 +193,16 @@
     <child link="imu_link" />
   </joint>
+  <link name="mid_mount" />
+  <joint name="mid_mount_joint" type="fixed">
+    <parent link="base_link" />
+    <child link="mid_mount" />
+    <origin xyz="0 0 ${deck_height}" rpy="0 0 0"/>
+  </joint>
   <!-- Bring in simulation data for Gazebo. -->
-  <xacro:include filename="ridgeback.gazebo" />
+  <xacro:include filename="$(find ridgeback_description)/urdf/ridgeback.gazebo" />
   <!-- Optional standard accessories, including their simulation data. The rendering
        of these into the final description is controlled by optenv variables, which
        default each one to off.-->
-  <xacro:include filename="accessories.urdf.xacro" />
+  <xacro:include filename="$(find ridgeback_description)/urdf/accessories.urdf.xacro" />
   <!-- Optional custom includes. -->
   <!--<xacro:include filename="$(optenv RIDGEBACK_URDF_EXTRAS empty.urdf)" />-->

Commit message: Added Sick S300 laser and Microstrain IMU upgrade accessories.

File: ridgeback_description/urdf/accessories.urdf.xacro (robot description, xacro)
@@ -14,24 +14,47 @@
   <xacro:if value="$(optenv RIDGEBACK_FRONT_HOKUYO_LASER 0)">
     <xacro:hokuyo_ust-10lx_mount prefix="front"
-                            topic="front/scan"
-                            location="1" />
+                                 topic="front/scan"
+                                 location="1" />
   </xacro:if>
   <!-- If enabled, generate the rear HOKUYO UST-10LX LASER payload. -->
   <xacro:if value="$(optenv RIDGEBACK_REAR_HOKUYO_LASER 0)">
     <xacro:hokuyo_ust-10lx_mount prefix="rear"
-                            topic="rear/scan"
-                            location="-1" />
+                                 topic="rear/scan"
+                                 location="-1" />
   </xacro:if>
   <!-- If enabled, generate the front SICK LMS111 LASER payload. -->
   <xacro:if value="$(optenv RIDGEBACK_FRONT_SICK_LASER 0)">
     <xacro:sick_lms1xx_mount prefix="front"
-                            topic="front/scan"
-                            location="1" />
+                             topic="front/scan"
+                             location="1" />
   </xacro:if>
   <!-- If enabled, generate the rear SICK LMS111 LASER payload. -->
   <xacro:if value="$(optenv RIDGEBACK_REAR_SICK_LASER 0)">
     <xacro:sick_lms1xx_mount prefix="rear"
-                            topic="rear/scan"
-                            location="-1" />
+                             topic="rear/scan"
+                             location="-1" />
+  </xacro:if>
+  <!-- If enabled, generate the front SICK S300 LASER payload.
+       This uses the same mesh as the lms1xx since they are the footprint
+       and the simulation parameters can be variable. -->
+  <xacro:if value="$(optenv RIDGEBACK_FRONT_S300_LASER 0)">
+    <xacro:sick_lms1xx_mount prefix="front"
+                             topic="front/scan"
+                             location="1" />
+  </xacro:if>
+  <!-- If enabled, generate the rear SICK S300 LASER payload. -->
+  <xacro:if value="$(optenv RIDGEBACK_REAR_S300_LASER 0)">
+    <xacro:sick_lms1xx_mount prefix="rear"
+                             topic="rear/scan"
+                             location="-1" />
+  </xacro:if>
+  <!-- If enabled, generate the optional Microstrain 3DM-GX2/3 IMU payload. -->
+  <xacro:include filename="$(find ridgeback_description)/urdf/accessories/microstrain_imu.urdf.xacro" />
+  <xacro:if value="$(optenv RIDGEBACK_MICROSTRAIN_IMU 0)">
+    <xacro:microstrain_imu prefix="$(optenv RIDGEBACK_MICROSTRAIN_IMU_PREFIX upgraded)"
+                           mount_link="$(optenv RIDGEBACK_MICROSTRAIN_IMU_MOUNT mid)_mount" >
+      <origin xyz="$(optenv RIDGEBACK_MICROSTRAIN_IMU_OFFSET 0 0 0)"
+              rpy="$(optenv RIDGEBACK_MICROSTRAIN_IMU_RPY 0 0 0)" />
+    </xacro:microstrain_imu>
   </xacro:if>
 </robot>

Commit message: Used sick-s300 xacro for simulation.

File: ridgeback_description/urdf/accessories.urdf.xacro (robot description, xacro)
@@ -10,4 +10,5 @@
   -->
   <xacro:include filename="$(find ridgeback_description)/urdf/accessories/sick_lms1xx_mount.urdf.xacro" />
+  <xacro:include filename="$(find ridgeback_description)/urdf/accessories/sick_s300_mount.urdf.xacro" />
   <xacro:include filename="$(find ridgeback_description)/urdf/accessories/hokuyo_ust-10lx_mount.urdf.xacro" />
   <!-- If enabled, generate the front HOKUYO UST-10LX LASER payload. -->
@@ -39,5 +40,5 @@
        and the simulation parameters can be variable. -->
   <xacro:if value="$(optenv RIDGEBACK_FRONT_S300_LASER 0)">
-    <xacro:sick_lms1xx_mount prefix="front"
+    <xacro:sick_s300_mount prefix="front"
                              topic="front/scan"
                              location="1" />
@@ -45,5 +46,5 @@
   <!-- If enabled, generate the rear SICK S300 LASER payload. -->
   <xacro:if value="$(optenv RIDGEBACK_REAR_S300_LASER 0)">
-    <xacro:sick_lms1xx_mount prefix="rear"
+    <xacro:sick_s300_mount prefix="rear"
                              topic="rear/scan"
                              location="-1" />

File: ridgeback_description/urdf/accessories/sick_s300_mount.urdf.xacro (robot description, xacro)
@@ -26,6 +26,6 @@
 <robot xmlns:xacro="http://ros.org/wiki/xacro">
   <xacro:include filename="$(find lms1xx)/urdf/sick_lms1xx.urdf.xacro" />
-  <xacro:macro name="sick_lms1xx_mount" params="prefix topic location">
-    <xacro:sick_lms1xx frame="${prefix}_laser" topic="${topic} update_rate="12.5" />
+  <xacro:macro name="sick_s300_mount" params="prefix topic location">
+    <xacro:sick_lms1xx frame="${prefix}_laser" topic="${topic}" update_rate="12.5" />
     <joint name="${prefix}_laser_joint" type="fixed">
       <!-- This offset is from the base of the bracket to the LIDAR's focal point. -->
@@ -35,3 +35,3 @@
     </joint>
   </xacro:macro>
-</robot>s
+</robot>

Commit message: Replace microstrain_3dmgx2_imu with microstrain_inertial_driver

File: ridgeback_description/urdf/accessories.urdf.xacro (robot description, xacro)
@@ -50,12 +50,19 @@
                              location="-1" />
   </xacro:if>
-  <!-- If enabled, generate the optional Microstrain 3DM-GX2/3 IMU payload. -->
-  <xacro:include filename="$(find ridgeback_description)/urdf/accessories/microstrain_imu.urdf.xacro" />
-  <xacro:if value="$(optenv RIDGEBACK_MICROSTRAIN_IMU 0)">
-    <xacro:microstrain_imu prefix="$(optenv RIDGEBACK_MICROSTRAIN_IMU_PREFIX upgraded)"
-                           mount_link="$(optenv RIDGEBACK_MICROSTRAIN_IMU_MOUNT mid)_mount" >
-      <origin xyz="$(optenv RIDGEBACK_MICROSTRAIN_IMU_OFFSET 0 0 0)"
-              rpy="$(optenv RIDGEBACK_MICROSTRAIN_IMU_RPY 0 0 0)" />
-    </xacro:microstrain_imu>
+  <!--
+    Add Microstrain IMU. By default the RIDGEBACK comes equipped with an IMU linked to "imu_link". These extra
+    optional microstrain IMU's will be added to another frame, by default, "microstrain_link".
+  -->
+  <xacro:if value="$(optenv RIDGEBACK_IMU_MICROSTRAIN 0)">
+    <xacro:property name="frame"  value="$(optenv RIDGEBACK_IMU_MICROSTRAIN_LINK microstrain_link)"/>
+    <xacro:property name="parent" value="$(optenv RIDGEBACK_IMU_MICROSTRAIN_PARENT imu_link)"/>
+    <xacro:property name="xyz"    value="$(optenv RIDGEBACK_IMU_MICROSTRAIN_OFFSET 0 0 0)"/>
+    <xacro:property name="rpy"    value="$(optenv RIDGEBACK_IMU_MICROSTRAIN_RPY 0 0 0)"/>
+    <link name="${frame}" />
+    <joint name="${frame}_joint" type="fixed">
+      <parent link="${parent}" />
+      <child link="${frame}" />
+      <origin xyz="${xyz}" rpy="${rpy}" />
+    </joint>
   </xacro:if>
 </robot>

Commit message: Update RIDGEBACK_IMU_MICROSTRAIN_OFFSET to RIDGEBACK_IMU_MICROSTRAIN_XYZ

File: ridgeback_description/urdf/accessories.urdf.xacro (robot description, xacro)
@@ -57,5 +57,5 @@
     <xacro:property name="frame"  value="$(optenv RIDGEBACK_IMU_MICROSTRAIN_LINK microstrain_link)"/>
     <xacro:property name="parent" value="$(optenv RIDGEBACK_IMU_MICROSTRAIN_PARENT imu_link)"/>
-    <xacro:property name="xyz"    value="$(optenv RIDGEBACK_IMU_MICROSTRAIN_OFFSET 0 0 0)"/>
+    <xacro:property name="xyz"    value="$(optenv RIDGEBACK_IMU_MICROSTRAIN_XYZ 0 0 0)"/>
     <xacro:property name="rpy"    value="$(optenv RIDGEBACK_IMU_MICROSTRAIN_RPY 0 0 0)"/>
     <link name="${frame}" />

Commit message: Revert "Update RIDGEBACK_IMU_MICROSTRAIN_OFFSET to RIDGEBACK_IMU_MICROSTRAIN_XYZ"
This reverts commit a23e11f2a1e03ed8dfef5eb2611055adf936a544.

File: ridgeback_description/urdf/accessories.urdf.xacro (robot description, xacro)
@@ -57,5 +57,5 @@
     <xacro:property name="frame"  value="$(optenv RIDGEBACK_IMU_MICROSTRAIN_LINK microstrain_link)"/>
     <xacro:property name="parent" value="$(optenv RIDGEBACK_IMU_MICROSTRAIN_PARENT imu_link)"/>
-    <xacro:property name="xyz"    value="$(optenv RIDGEBACK_IMU_MICROSTRAIN_XYZ 0 0 0)"/>
+    <xacro:property name="xyz"    value="$(optenv RIDGEBACK_IMU_MICROSTRAIN_OFFSET 0 0 0)"/>
     <xacro:property name="rpy"    value="$(optenv RIDGEBACK_IMU_MICROSTRAIN_RPY 0 0 0)"/>
     <link name="${frame}" />

Commit message: Add URDF link and joint for microstrain_inertial_driver Microstrain IMU.

File: ridgeback_description/urdf/accessories.urdf.xacro (robot description, xacro)
@@ -59,3 +59,19 @@
     </xacro:microstrain_imu>
   </xacro:if>
+  <!--
+    Add Microstrain IMU. By default the Ridgeback comes equipped with an IMU linked to "imu_link". These extra
+    optional microstrain IMU's will be added to another frame, by default, "microstrain_link".
+  -->
+  <xacro:if value="$(optenv RIDGEBACK_IMU_MICROSTRAIN 0)">
+    <xacro:property name="frame"  value="$(optenv RIDGEBACK_IMU_MICROSTRAIN_LINK microstrain_link)"/>
+    <xacro:property name="parent" value="$(optenv RIDGEBACK_IMU_MICROSTRAIN_PARENT base_link)"/>
+    <xacro:property name="xyz"    value="$(optenv RIDGEBACK_IMU_MICROSTRAIN_OFFSET -0.139 0.096 0.100)"/>
+    <xacro:property name="rpy"    value="$(optenv RIDGEBACK_IMU_MICROSTRAIN_RPY ${PI} 0 -${PI/2})"/>
+    <link name="${frame}" />
+    <joint name="${frame}_joint" type="fixed">
+      <parent link="${parent}" />
+      <child link="${frame}" />
+      <origin xyz="${xyz}" rpy="${rpy}" />
+    </joint>
+  </xacro:if>
 </robot>
